File: PCB/v1/v1.kicad_pcb (KiCad board)
At the start: 2 copper layers, 13 x 17.4 mm, 3 parts, among them P1 USB_C_Plug_USB2.0

Commit message: Changes to PCB
Routing:
- net VBUS: track 0.28 -> 7.32 mm, vias 0 -> 1
Changed lines of the file:
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@@
 			(at -5.225 3.5 180)
 			(size 1.2 2.23)
-			(drill oval 0.5 1.53)
+			(drill oval 0.5 1.53
+				(offset -0.2 0)
+			)
 			(layers "*.Cu" "*.Mask")
 			(remove_unused_layers no)
-			(roundrect_rratio 0.5)
+			(roundrect_rratio 0.2083333333)
 			(net 3 "GND")
 			(pinfunction "SHIELD")
@@
 			(at 5.225 3.5 180)
 			(size 1.2 2.23)
-			(drill oval 0.5 1.53)
+			(drill oval 0.5 1.53
+				(offset 0.2 0)
+			)
 			(layers "*.Cu" "*.Mask")
 			(remove_unused_layers no)
-			(roundrect_rratio 0.5)
+			(roundrect_rratio 0.2083333333)
 			(net 3 "GND")
 			(pinfunction "SHIELD")
@@
 			)
 		)
-		(pad "1" thru_hole roundrect
-			(at -2.6 6.75 180)
+		(pad "1" smd roundrect
+			(at -2.6 6.65 180)
 			(size 2.6 1.5)
-			(drill oval 1.8 1)
-			(layers "*.Cu" "*.Mask")
-			(remove_unused_layers no)
+			(layers "F.Cu" "F.Mask" "F.Paste")
 			(roundrect_rratio 0.15)
 			(net 3 "GND")
 		)
-		(pad "1" thru_hole roundrect
-			(at -2.6 14.15 180)
+		(pad "1" smd roundrect
+			(at -2.6 14.25 180)
 			(size 2.6 1.5)
-			(drill oval 1.8 1)
-			(layers "*.Cu" "*.Mask")
-			(remove_unused_layers no)
+			(layers "F.Cu" "F.Mask" "F.Paste")
 			(roundrect_rratio 0.15)
 			(net 3 "GND")
 		)
-		(pad "1" thru_hole roundrect
-			(at 2.6 6.75 180)
+		(pad "1" smd roundrect
+			(at 2.6 6.65 180)
 			(size 2.6 1.5)
-			(drill oval 1.8 1)
-			(layers "*.Cu" "*.Mask")
-			(remove_unused_layers no)
+			(layers "F.Cu" "F.Mask" "F.Paste")
 			(roundrect_rratio 0.15)
 			(net 3 "GND")
 		)
-		(pad "1" thru_hole roundrect
-			(at 2.6 14.15 180)
+		(pad "1" smd roundrect
+			(at 2.6 14.25 180)
 			(size 2.6 1.5)
-			(drill oval 1.8 1)
-			(layers "*.Cu" "*.Mask")
-			(remove_unused_layers no)
+			(layers "F.Cu" "F.Mask" "F.Paste")
 			(roundrect_rratio 0.15)
 			(net 3 "GND")
@@
 	)
 	(segment
-		(start 104 62.71)
+		(start 104 62.21)
 		(end 104 61.81)
 		(width 0.2)
@@
 	)
 	(via
-		(at 104 62.71)
+		(at 104 62.21)
 		(size 0.6)
 		(drill 0.3)
@@
 	)
 	(segment
+		(start 104 62.21)
+		(end 104 62.71)
+		(width 0.2)
+		(layer "B.Cu")
+		(net 2)
+	)
+	(segment
+		(start 104 62.71)
+		(end 103.91 62.8)
+		(width 0.2)
+		(layer "B.Cu")
+		(net 2)
+	)
+	(segment
 		(start 103.91 62.8)
 		(end 103.91 63.91)
-		(width 0.2)
-		(layer "B.Cu")
-		(net 2)
-	)
-	(segment
-		(start 104 62.71)
-		(end 103.91 62.8)
 		(width 0.2)
 		(layer "B.Cu")
@@
 	)
 	(segment
+		(start 108 62.01)
+		(end 107.16 61.17)
+		(width 0.2)
+		(layer "F.Cu")
+		(net 5)
+	)
+	(segment
+		(start 107.16 61.17)
+		(end 107.16 60.44)
+		(width 0.2)
+		(layer "F.Cu")
+		(net 5)
+	)
+	(via
+		(at 108 62.01)
+		(size 0.6)
+		(drill 0.3)
+		(layers "F.Cu" "B.Cu")
+		(net 5)
+	)
+	(segment
 		(start 107.69 66.235)
 		(end 107.975 66.235)
 		(width 0.2)
 		(layer "B.Cu")
+		(net 5)
+	)
+	(segment
+		(start 108.916 62.926)
+		(end 108 62.01)
+		(width 0.2)
+		(layer "B.Cu")
+		(net 5)
+	)
+	(segment
+		(start 108.916 65.009)
+		(end 108.916 62.926)
+		(width 0.2)
+		(layer "B.Cu")
+		(net 5)
+	)
+	(segment
+		(start 107.69 66.235)
+		(end 108.916 65.009)
+		(width 0.2)
+		(layer "B.Cu")
